Commit message: Added thymio urdf

File: urdf/thymio_simple.urdf.xacro (robot description, xacro)
@@ -17,5 +17,5 @@
     <link name="base_link">
         <visual>
-            <origin xyz="0 0 0"/>
+            <origin xyz="0 0 0.0225"/>
             <geometry>
                 <box size="0.11 0.112 0.045"/>
@@ -24,14 +24,78 @@
         </visual>
         <collision>
-            <origin xyz="0 0 0"/>
+            <origin xyz="0 0 0.0225"/>
             <geometry>
                 <box size="0.11 0.112 0.045"/>
             </geometry>
+        </collision>
+        <inertial>
+            <mass value = "0.270"/>
+            <xacro:box_inertia mass="0.270" x="0.11" y="0.112" z="0.045"/>
+        </inertial>
+        <!-- Implement the caster wheel -->
+        <visual>
+            <origin xyz="0 0.04 0"/>
+            <geometry>
+                <sphere radius="0.01"/>
+            </geometry>
             <material name="white"/>
+        </visual>
+        <collision>
+            <origin xyz="0 0.04 0"/>
+            <geometry>
+                <sphere radius="0.01"/>
+            </geometry>
         </collision>
-        <!-- Implement the caster wheel -->
     </link>
+    <joint name="right_joint" type="continuous">
+        <parent link="base_link"/>
+        <child link="right_wheel_link"/>
+        <axis rpy="0 0 0" xyz="0 1 0"/>
+        <origin xyz="0.05 -0.02 0.01"/>
+    </joint>
     <!-- Implement the left wheel -->
     <!-- Implement the joint for the left wheel -->
+    <link name="right_wheel_link">
+        <visual>
+            <origin xyz="0 0 0" rpy="1.57 0 1.57"/>
+        <geometry>
+            <cylinder length="0.01" radius="0.02"/>
+        </geometry>
+        </visual>
+        <collision>
+            <origin xyz="0 0 0" rpy="1.57 0 1.57"/>
+            <geometry>
+                <cylinder length="0.01" radius="0.02"/>
+            </geometry>
+        </collision>
+        <inertial>
+            <mass value = "0.08"/>
+            <xacro:cylinder_inertia mass="0.08" h="0.01" r="0.02"/>
+        </inertial>
+    </link>
+    <joint name="left_joint" type="continuous">
+        <parent link="base_link"/>
+        <child link="left_wheel_link"/>
+        <axis rpy="0 0 0" xyz="0 1 0"/>
+        <origin xyz="-0.05 -0.02 0.01"/>
+    </joint>
+    <link name="left_wheel_link">
+        <visual>
+            <origin xyz="0 0 0" rpy="1.57 0 1.57"/>
+        <geometry>
+            <cylinder length="0.01" radius="0.02"/>
+        </geometry>
+        </visual>
+        <collision>
+            <origin xyz="0 0 0" rpy="1.57 0 1.57"/>
+            <geometry>
+                <cylinder length="0.01" radius="0.02"/>
+            </geometry>
+        </collision>
+        <inertial>
+            <mass value = "0.08"/>
+            <xacro:cylinder_inertia mass="0.08" h="0.01" r="0.02"/>
+        </inertial>
+    </link>
     <!-- Implement the right wheel -->
     <!-- Implement the joint for the right wheel -->

Commit message: Fix wrong joint name

File: urdf/thymio_simple.urdf.xacro (robot description, xacro)
@@ -48,5 +48,7 @@
         </collision>
     </link>
-    <joint name="right_joint" type="continuous">
+    <!-- Implement the right wheel -->
+    <!-- Implement the joint for the right wheel -->
+    <joint name="right_wheel_joint" type="continuous">
         <parent link="base_link"/>
         <child link="right_wheel_link"/>
@@ -54,6 +56,4 @@
         <origin xyz="0.05 -0.02 0.01"/>
     </joint>
-    <!-- Implement the left wheel -->
-    <!-- Implement the joint for the left wheel -->
     <link name="right_wheel_link">
         <visual>
@@ -74,5 +74,7 @@
         </inertial>
     </link>
-    <joint name="left_joint" type="continuous">
+    <!-- Implement the left wheel -->
+    <!-- Implement the joint for the left wheel -->
+    <joint name="left_wheel_joint" type="continuous">
         <parent link="base_link"/>
         <child link="left_wheel_link"/>
@@ -98,6 +100,4 @@
         </inertial>
     </link>
-    <!-- Implement the right wheel -->
-    <!-- Implement the joint for the right wheel -->
     <!-- Add your sensors using the macro -->
 </robot>

Commit message: Fix axis alignment and corrected wheel size

File: urdf/thymio_simple.urdf.xacro (robot description, xacro)
@@ -30,10 +30,10 @@
         </collision>
         <inertial>
-            <mass value = "0.270"/>
-            <xacro:box_inertia mass="0.270" x="0.11" y="0.112" z="0.045"/>
+            <mass value = "${body_mass}"/>
+            <xacro:box_inertia mass="${body_mass}" x="0.11" y="0.112" z="0.045"/>
         </inertial>
         <!-- Implement the caster wheel -->
         <visual>
-            <origin xyz="0 0.04 0"/>
+            <origin xyz="0.035 0 0"/>
             <geometry>
                 <sphere radius="0.01"/>
@@ -42,5 +42,5 @@
         </visual>
         <collision>
-            <origin xyz="0 0.04 0"/>
+            <origin xyz="0.035 0 0"/>
             <geometry>
                 <sphere radius="0.01"/>
@@ -54,22 +54,22 @@
         <child link="right_wheel_link"/>
         <axis rpy="0 0 0" xyz="0 1 0"/>
-        <origin xyz="0.05 -0.02 0.01"/>
+        <origin xyz="-0.02 -0.0551 0.01"/>
     </joint>
     <link name="right_wheel_link">
         <visual>
-            <origin xyz="0 0 0" rpy="1.57 0 1.57"/>
+            <origin xyz="0 0 0" rpy="1.5707 0 0"/>
         <geometry>
-            <cylinder length="0.01" radius="0.02"/>
+            <cylinder length="${wheel_len}" radius="${wheel_radius}"/>
         </geometry>
         </visual>
         <collision>
-            <origin xyz="0 0 0" rpy="1.57 0 1.57"/>
+            <origin xyz="0 0 0" rpy="1.5707 0 0"/>
             <geometry>
-                <cylinder length="0.01" radius="0.02"/>
+                <cylinder length="${wheel_len}" radius="${wheel_radius}"/>
             </geometry>
         </collision>
         <inertial>
-            <mass value = "0.08"/>
-            <xacro:cylinder_inertia mass="0.08" h="0.01" r="0.02"/>
+            <mass value = "${wheel_mass}"/>
+            <xacro:cylinder_inertia mass="${wheel_mass}" h="${wheel_len}" r="${wheel_radius}"/>
         </inertial>
     </link>
@@ -80,22 +80,22 @@
         <child link="left_wheel_link"/>
         <axis rpy="0 0 0" xyz="0 1 0"/>
-        <origin xyz="-0.05 -0.02 0.01"/>
+        <origin xyz="-0.02 0.0551  0.01"/>
     </joint>
     <link name="left_wheel_link">
         <visual>
-            <origin xyz="0 0 0" rpy="1.57 0 1.57"/>
+            <origin xyz="0 0 0" rpy="1.5707 0 0"/>
         <geometry>
-            <cylinder length="0.01" radius="0.02"/>
+            <cylinder length="${wheel_len}" radius="${wheel_radius}"/>
         </geometry>
         </visual>
         <collision>
-            <origin xyz="0 0 0" rpy="1.57 0 1.57"/>
+            <origin xyz="0 0 0" rpy="1.5707 0 0"/>
             <geometry>
-                <cylinder length="0.01" radius="0.02"/>
+                <cylinder length="${wheel_len}" radius="${wheel_radius}"/>
             </geometry>
         </collision>
         <inertial>
-            <mass value = "0.08"/>
-            <xacro:cylinder_inertia mass="0.08" h="0.01" r="0.02"/>
+            <mass value = "${wheel_mass}"/>
+            <xacro:cylinder_inertia mass="${wheel_mass}" h="${wheel_len}" r="${wheel_radius}"/>
         </inertial>
     </link>

Commit message: Added final controller and urdf

File: urdf/thymio_simple.urdf.xacro (robot description, xacro)
@@ -33,5 +33,5 @@
             <xacro:box_inertia mass="${body_mass}" x="0.11" y="0.112" z="0.045"/>
         </inertial>
-        <!-- Implement the caster wheel -->
+        <!-- Caster wheel -->
         <visual>
             <origin xyz="0.035 0 0"/>
@@ -48,11 +48,11 @@
         </collision>
     </link>
-    <!-- Implement the right wheel -->
-    <!-- Implement the joint for the right wheel -->
+    <!-- Right wheel -->
+    <!-- Joint for the right wheel -->
     <joint name="right_wheel_joint" type="continuous">
         <parent link="base_link"/>
         <child link="right_wheel_link"/>
         <axis rpy="0 0 0" xyz="0 1 0"/>
-        <origin xyz="-0.02 -0.0551 0.01"/>
+        <origin xyz="-0.02 -0.0476 0.01"/>
     </joint>
     <link name="right_wheel_link">
@@ -74,11 +74,11 @@
         </inertial>
     </link>
-    <!-- Implement the left wheel -->
-    <!-- Implement the joint for the left wheel -->
+    <!-- Left wheel -->
+    <!-- Joint for the left wheel -->
     <joint name="left_wheel_joint" type="continuous">
         <parent link="base_link"/>
         <child link="left_wheel_link"/>
         <axis rpy="0 0 0" xyz="0 1 0"/>
-        <origin xyz="-0.02 0.0551  0.01"/>
+        <origin xyz="-0.02 0.0476  0.01"/>
     </joint>
     <link name="left_wheel_link">
@@ -100,4 +100,11 @@
         </inertial>
     </link>
-    <!-- Add your sensors using the macro -->
+    <!-- Sensors-->
+    <xacro:csensor plink="base_link" id="0" mass="0.001" originrpy="0 0 0" originxyz="0 0 0" jointxyz="0.055 0.055 0.0225" jointrpy="0 0 -0.73" />
+    <xacro:csensor plink="base_link" id="1" mass="0.001" originrpy="0 0 0" originxyz="0 0 0" jointxyz="0.0685 0.0307 0.0225" jointrpy="0 0 -1.15" />
+    <xacro:csensor plink="base_link" id="2" mass="0.001" originrpy="0 0 0" originxyz="0 0 0" jointxyz="0.0751 0 0.0225" jointrpy="0 0 -1.57" />
+    <xacro:csensor plink="base_link" id="3" mass="0.001" originrpy="0 0 0" originxyz="0 0 0" jointxyz="0.0685 -0.0307 0.0225" jointrpy="0 0 -1.99" />
+    <xacro:csensor plink="base_link" id="4" mass="0.001" originrpy="0 0 0" originxyz="0 0 0" jointxyz="0.055 -0.055 0.0225" jointrpy="0 0 -2.41" />
+    <xacro:csensor plink="base_link" id="5" mass="0.001" originrpy="0 0 0" originxyz="0 0 0" jointxyz="-0.055 0.045 0.0225" jointrpy="0 0 1.57" />
+    <xacro:csensor plink="base_link" id="6" mass="0.001" originrpy="0 0 0" originxyz="0 0 0" jointxyz="-0.055 -0.045 0.0225" jointrpy="0 0 1.57" />
 </robot>
